Commit message: Fulfill the simple simumation in Gazebo

File: src/node_pkg/urdf/robot_description.urdf (robot description, URDF)
Before this commit: robot view_robot_pkg, 9 links, 8 joints
Links:
- link base_link: geometry collision mesh filename=package://node_pkg/meshes/base_link.STL; visual mesh filename=package://node_pkg/meshes/base_link.STL
- link left_casterwheel_after_Link: geometry collision mesh filename=package://node_pkg/meshes/left_casterwheel_after_Link.STL; visual mesh filename=package://node_pkg/meshes/left_casterwheel_after_Link.STL
- link left_casterwheel_before_Link: geometry collision mesh filename=package://node_pkg/meshes/left_casterwheel_before_Link.STL; visual mesh filename=package://node_pkg/meshes/left_casterwheel_before_Link.STL
- link leftwheel_Link: geometry collision mesh filename=package://node_pkg/meshes/leftwheel_Link.STL; visual mesh filename=package://node_pkg/meshes/leftwheel_Link.STL
- link lidar_link: geometry collision mesh filename=package://node_pkg/meshes/lidar_Link.STL; visual mesh filename=package://node_pkg/meshes/lidar_Link.STL
- link right_casterwheel_after_Link: geometry collision mesh filename=package://node_pkg/meshes/right_casterwheel_after_Link.STL; visual mesh filename=package://node_pkg/meshes/right_casterwheel_after_Link.STL
- link right_casterwheel_before_Link: geometry collision mesh filename=package://node_pkg/meshes/right_casterwheel_before_Link.STL; visual mesh filename=package://node_pkg/meshes/right_casterwheel_before_Link.STL
- link rightwheel_Link: geometry collision mesh filename=package://node_pkg/meshes/rightwheel_Link.STL; visual mesh filename=package://node_pkg/meshes/rightwheel_Link.STL

Commit message: added robot-tracking-human feature

File: src/node_pkg/urdf/robot_description.urdf (robot description, URDF)
Before this commit: robot node_pkg, 9 links, 8 joints
Links:
- added link camera_link, mass 0.1; collision box size=0.03 0.08 0.03; visual box size=0.03 0.08 0.03
Joints:
- added joint camera_joint: type fixed, parent base_link, child camera_link, origin xyz=0.15 0 0.05 rpy=0 0 0
